File: oal-psu.kicad_pcb (KiCad board)
At the start: 2 copper layers, 0 parts

Commit message: initial layout work
Parts:
- added C101: 0.1uF, ose-audio-labs:TDK-B32529-63VAC, F.Cu at (135.5, 79.5)
- added C102: 0.01uF, ose-audio-labs:TDK-B32529-63VAC, F.Cu at (142.0, 79.5)
- added C103: 1kuF, ose-audio-labs:35V-LYTIC-7.5-5, F.Cu at (187.0, 80.0)
- added C104: 1kuF, ose-audio-labs:35V-LYTIC-7.5-5, F.Cu at (187.0, 98.5)
- added C105: 1kuF, ose-audio-labs:35V-LYTIC-7.5-5-10snap, F.Cu at (170.8, 89.2)
- added C106: 1kuF, ose-audio-labs:35V-LYTIC-7.5-5, F.Cu at (154.5, 98.5)
- added C107: 1kuF, ose-audio-labs:35V-LYTIC-7.5-5, F.Cu at (154.5, 80.0)
- added C108: 47uF, Capacitors_Tantalum_SMD:TantalC_SizeD_EIA-7343_Reflow, F.Cu at (198.9, 89.1)
- added C109: 10uF, Capacitors_SMD:C_1206, F.Cu at (209.0, 95.3)
- added C110: 1uF, Capacitors_SMD:C_0805, F.Cu at (207.5, 91.8)
- added C111: 10uF, Capacitors_SMD:C_1206, F.Cu at (215.0, 96.3)
- added C112: 10uF, Capacitors_SMD:C_1206, F.Cu at (215.0, 99.0)
- added C113: 10uF, Capacitors_SMD:C_1206, F.Cu at (215.0, 101.8)
- added C114: 10uF, Capacitors_SMD:C_1206, F.Cu at (215.0, 106.8)
- added C115: 10uF, Capacitors_SMD:C_1206, F.Cu at (215.0, 104.2)
- added C201: 0.1uF, ose-audio-labs:TDK-B32529-63VAC, F.Cu at (136.5, 143.0)
- added C202: 0.01uF, ose-audio-labs:TDK-B32529-63VAC, F.Cu at (136.5, 135.0)
- added C203: 1kuF, ose-audio-labs:35V-LYTIC-7.5-5, F.Cu at (140.2, 162.0)
- added C204: 1kuF, ose-audio-labs:35V-LYTIC-7.5-5, F.Cu at (151.2, 143.0)
- added C205: 1kuF, ose-audio-labs:35V-LYTIC-7.5-5, F.Cu at (177.2, 139.0)
- added C206: 1kuF, ose-audio-labs:35V-LYTIC-7.5-5, F.Cu at (195.8, 154.0)
- added C207: 1kuF, ose-audio-labs:35V-LYTIC-7.5-5-10snap, F.Cu at (167.0, 163.0)
- added C208: 47uF, Capacitors_Tantalum_SMD:TantalC_SizeD_EIA-7343_Reflow, F.Cu at (162.0, 133.0)
- added C209: 10uF, Capacitors_SMD:C_1206, F.Cu at (169.0, 126.0)
- added C210: 1uF, Capacitors_SMD:C_0805, F.Cu at (221.0, 149.0)
- added C211: 10uF, Capacitors_SMD:C_1206, F.Cu at (220.5, 143.0)
- added C212: 10uF, Capacitors_SMD:C_1206, F.Cu at (227.5, 149.0)
- added C213: 10uF, Capacitors_SMD:C_1206, F.Cu at (227.5, 144.0)
- added C214: 10uF, Capacitors_SMD:C_1206, F.Cu at (234.5, 153.0)
- added C215: 10uF, Capacitors_SMD:C_1206, F.Cu at (233.5, 146.0)
- added D101: DIODE-45, ose-audio-labs:DO-221AC, F.Cu at (140.5, 95.3)
- added D102: DIODE-45, ose-audio-labs:DO-221AC, F.Cu at (134.5, 95.3)
- added D103: DIODE-45, ose-audio-labs:DO-221AC, F.Cu at (140.5, 102.3)
- added D104: DIODE-45, ose-audio-labs:DO-221AC, F.Cu at (134.5, 102.3)
- added D201: DIODE-45, ose-audio-labs:DO-221AC, F.Cu at (135.8, 127.0)
- added D202: DIODE-45, ose-audio-labs:DO-221AC, F.Cu at (147.0, 126.0)
- added D203: DIODE-45, ose-audio-labs:DO-221AC, F.Cu at (137.0, 119.0)
- added D204: DIODE-45, ose-audio-labs:DO-221AC, F.Cu at (147.2, 119.0)
- added F1: FUSE, ose-audio-labs:LITTLEFUSE-0PTF0078P, F.Cu at (44.9, 110.0)
- added J1: MAINS_LINE, ose-audio-labs:PHEONIX_SPT_5-2POS, F.Cu at (40.6, 124.6)
- added J2: MAINS_NEUTRAL, ose-audio-labs:PHEONIX_SPT_5-2POS, F.Cu at (40.5, 138.0)
- added J3: OUTPUT, ose-audio-labs:PHEONIX_MC1.5-12-G-3.5, F.Cu at (227.6, 110.2)
- added LED101: LED, LEDs:LED-1206, F.Cu at (220.9, 96.5)
- added LED201: LED, LEDs:LED-1206, F.Cu at (202.6, 137.0)
- added P101: ENABLE_A, Pin_Headers:Pin_Header_Straight_1x02, F.Cu at (202.5, 80.5)
- added P2: OUTPUT_SELECT, Pin_Headers:Pin_Header_Straight_2x03, F.Cu at (220.8, 107.9)
- added P201: ENABLE_B, Pin_Headers:Pin_Header_Straight_1x02, F.Cu at (185.0, 126.5)
- added R101: R, Resistors_SMD:R_1210, F.Cu at (140.6, 86.5)
- added R102: 820R, Resistors_SMD:R_0805, F.Cu at (222.5, 93.2)
- added R201: R, Resistors_SMD:R_1210, F.Cu at (143.6, 133.0)
- added R202: 820R, Resistors_SMD:R_0805, F.Cu at (202.1, 145.0)
- added SW1: DPDT_SLIDE, ose-audio-labs:CK_V80212MS02Q-VOLTAGE_SELECTOR, F.Cu at (46.3, 88.3)
- added SW102: VOLTAGE_A, ose-audio-labs:DIP8-HALF-PITCH, F.Cu at (213.6, 80.9)
- added SW202: VOLTAGE_B, ose-audio-labs:DIP8-HALF-PITCH, F.Cu at (195.6, 126.9)
- added T1: TALEMA 15/25VA, ose-audio-labs:TALEMA_70000K_35VA, F.Cu at (95.0, 110.0)
- added U101: TPS7A4700, PVQFN-N20-new, F.Cu at (214.2, 90.7)
- added U201: TPS7A4700, ose-audio-labs:PVQFN-N20, F.Cu at (213.7, 138.6)
Routing:
- net NEUTRAL: track 0.00 -> 116.3 mm
- net UNREG-A: track 0.00 -> 106.2 mm
- net ENABLE-A: track 0.00 -> 69.5 mm
- net Net-(F1-Pad2): track 0.00 -> 62.5 mm
- net Net-(SW1-Pad5): track 0.00 -> 61.1 mm
- net Net-(C101-Pad2): track 0.00 -> 44.8 mm
- net NEG-A: track 0.00 -> 44.7 mm
- net LINE: track 0.00 -> 39.7 mm
- net Net-(C101-Pad1): track 0.00 -> 37.2 mm
- net SENSE-A: track 0.00 -> 29.0 mm
- net Net-(SW1-Pad2): track 0.00 -> 13.2 mm
- net Net-(SW1-Pad3): track 0.00 -> 8.00 mm
- net Net-(SW102-Pad1): track 0.00 -> 7.61 mm
- net Net-(SW102-Pad8): track 0.00 -> 7.06 mm
- net Net-(SW102-Pad2): track 0.00 -> 6.12 mm
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- added copper zone on B.Cu, net NEG-A
- added copper zone on F.Cu, net NEG-A
- added copper zone on F.Cu, net POS-A
- added copper zone on F.Cu, net UNREG-A
Other:
- net class Default: clearance 0.2 -> 0.3; trace_width 0.25 -> 0.7
- net class LOW_VOLTAGE added: clearance 0.3, trace_width 0.3, via_dia 0.6, via_drill 0.4
- net class MAINS added: clearance 1.85, trace_width 3, via_dia 0.6, via_drill 0.4
- rule trace_clearance: 0.2 -> 0.3

Commit message: board outline
Parts:
- moved F1 0.80 mm to (45.7, 110.0)
Routing:
- net Net-(SW1-Pad5): track 61.1 -> 70.4 mm
- net Net-(F1-Pad2): track 62.5 -> 66.9 mm
- net NEUTRAL: track 116.3 -> 118.0 mm
Other:
- board outline added: 200 x 80 mm
- net class MAINS: trace_width 3 -> 2.28

Commit message: more cleanup
Parts:
- added REF**: MOUNTING_HOLE-M3, MOUNTING_HOLE-M3, F.Cu at (36.0, 146.0)
- added REF**: MOUNTING_HOLE-M3, MOUNTING_HOLE-M3, F.Cu at (228.0, 74.0)
- added REF**: MOUNTING_HOLE-M3, MOUNTING_HOLE-M3, F.Cu at (228.0, 146.0)
- added REF**: MOUNTING_HOLE-M3, MOUNTING_HOLE-M3, F.Cu at (36.0, 74.0)
- moved C210 32.3 mm to (212.0, 180.0)
- moved C211 32.3 mm to (211.5, 174.0)
- moved C212 32.3 mm to (218.5, 180.0)
- moved C213 32.3 mm to (218.5, 175.0)
- moved C214 32.3 mm to (225.5, 184.0)
- moved C215 32.3 mm to (224.5, 177.0)
Changed lines of the file:
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@@
     (links 202)
     (no_connects 87)
-    (area 17.000001 61.067238 244.100001 180.083297)
+    (area 31.749999 69.749999 232.250001 150.250001)
     (thickness 1.6)
     (drawings 7)
     (tracks 147)
     (zones 0)
-    (modules 57)
+    (modules 61)
     (nets 43)
   )
@@
   )
   (setup
-    (last_trace_width 3)
+    (last_trace_width 0.7)
     (user_trace_width 0.3)
     (user_trace_width 0.5)
@@
     (add_net "Net-(SW1-Pad5)")
   )
+  (module MOUNTING_HOLE-M3 (layer F.Cu)
+    (at 36 146)
+    (fp_text reference REF** (at 0 5) (layer F.SilkS) hide
+      (effects (font (size 1.5 1.5) (thickness 0.25)))
+    )
+    (fp_text value MOUNTING_HOLE-M3 (at 0 -5) (layer F.Fab)
+      (effects (font (size 1.5 1.5) (thickness 0.25)))
+    )
+    (fp_circle (center 0 0) (end 0 -3.3) (layer F.CrtYd) (width 0.2))
+    (pad 1 thru_hole circle (at 0 0) (size 7.3 7.3) (drill 3.1) (layers *.Cu *.Mask F.SilkS)
+      (zone_connect 0))
+  )
+  (module MOUNTING_HOLE-M3 (layer F.Cu)
+    (at 228 74)
+    (fp_text reference REF** (at 0 5) (layer F.SilkS) hide
+      (effects (font (size 1.5 1.5) (thickness 0.25)))
+    )
+    (fp_text value MOUNTING_HOLE-M3 (at 0 -5) (layer F.Fab)
+      (effects (font (size 1.5 1.5) (thickness 0.25)))
+    )
+    (fp_circle (center 0 0) (end 0 -3.3) (layer F.CrtYd) (width 0.2))
+    (pad 1 thru_hole circle (at 0 0) (size 7.3 7.3) (drill 3.1) (layers *.Cu *.Mask F.SilkS)
+      (zone_connect 0))
+  )
+  (module MOUNTING_HOLE-M3 (layer F.Cu)
+    (at 228 146)
+    (fp_text reference REF** (at 0 5) (layer F.SilkS) hide
+      (effects (font (size 1.5 1.5) (thickness 0.25)))
+    )
+    (fp_text value MOUNTING_HOLE-M3 (at 0 -5) (layer F.Fab)
+      (effects (font (size 1.5 1.5) (thickness 0.25)))
+    )
+    (fp_circle (center 0 0) (end 0 -3.3) (layer F.CrtYd) (width 0.2))
+    (pad 1 thru_hole circle (at 0 0) (size 7.3 7.3) (drill 3.1) (layers *.Cu *.Mask F.SilkS)
+      (zone_connect 0))
+  )
+  (module MOUNTING_HOLE-M3 (layer F.Cu)
+    (at 36 74)
+    (fp_text reference REF** (at 0 5) (layer F.SilkS) hide
+      (effects (font (size 1.5 1.5) (thickness 0.25)))
+    )
+    (fp_text value MOUNTING_HOLE-M3 (at 0 -5) (layer F.Fab)
+      (effects (font (size 1.5 1.5) (thickness 0.25)))
+    )
+    (fp_circle (center 0 0) (end 0 -3.3) (layer F.CrtYd) (width 0.2))
+    (pad 1 thru_hole circle (at 0 0) (size 7.3 7.3) (drill 3.1) (layers *.Cu *.Mask F.SilkS)
+      (zone_connect 0))
+  )
   (module PVQFN-N20-new (layer F.Cu)
     (at 214.19 90.65 180)
@@
   )
   (module Capacitors_SMD:C_0805 (layer F.Cu)
-    (at 221 149)
+    (at 212 180)
     (descr "Capacitor SMD 0805, reflow soldering, AVX (see smccp.pdf)")
     (tags "capacitor 0805")
@@
   )
   (module Capacitors_SMD:C_1206 (layer F.Cu)
-    (at 220.5 143)
+    (at 211.5 174)
     (descr "Capacitor SMD 1206, reflow soldering, AVX (see smccp.pdf)")
     (tags "capacitor 1206")
@@
   )
   (module Capacitors_SMD:C_1206 (layer F.Cu)
-    (at 227.5 149)
+    (at 218.5 180)
     (descr "Capacitor SMD 1206, reflow soldering, AVX (see smccp.pdf)")
     (tags "capacitor 1206")
@@
   )
   (module Capacitors_SMD:C_1206 (layer F.Cu)
-    (at 227.5 144)
+    (at 218.5 175)
     (descr "Capacitor SMD 1206, reflow soldering, AVX (see smccp.pdf)")
     (tags "capacitor 1206")
@@
   )
   (module Capacitors_SMD:C_1206 (layer F.Cu)
-    (at 234.5 153)
+    (at 225.5 184)
     (descr "Capacitor SMD 1206, reflow soldering, AVX (see smccp.pdf)")
     (tags "capacitor 1206")
@@
   )
   (module Capacitors_SMD:C_1206 (layer F.Cu)
-    (at 233.5 146)
+    (at 224.5 177)
     (descr "Capacitor SMD 1206, reflow soldering, AVX (see smccp.pdf)")
     (tags "capacitor 1206")
@@
   (segment (start 135.5 77) (end 142 77) (width 1.2) (layer B.Cu) (net 1) (status 30))
   (segment (start 128 77) (end 135.5 77) (width 1.2) (layer B.Cu) (net 1) (status 30))
-  (segment (start 135.5 82) (end 135.5 82.9) (width 0.7) (layer F.Cu) (net 2) (status 10))
-  (segment (start 135.5 82.9) (end 139.1 86.5) (width 0.7) (layer F.Cu) (net 2) (status 20))
+  (segment (start 135.5 82) (end 135.5 82.9) (width 0.7) (layer F.Cu) (net 2))
+  (segment (start 135.5 82.9) (end 139.1 86.5) (width 0.7) (layer F.Cu) (net 2))
   (segment (start 128 82.08) (end 128 98.16) (width 1.2) (layer F.Cu) (net 2) (status 10))
   (segment (start 128 98.16) (end 134.34 104.5) (width 1.2) (layer F.Cu) (net 2) (status 20))
@@
     (polygon
       (pts
-        (xy 145 70.5) (xy 145 110) (xy 230 109.75) (xy 230 70.5)
+        (xy 145 70.5) (xy 145 109.5) (xy 231.5 109.5) (xy 231.5 70.5)
       )
     )
@@
     (polygon
       (pts
-        (xy 145 70.5) (xy 145 110) (xy 198 110) (xy 198 70.5)
+        (xy 145 70.5) (xy 145 109.5) (xy 198 109.5) (xy 198 70.5)
       )
     )
@@
     (polygon
       (pts
-        (xy 199 70.5) (xy 230.25 70.5) (xy 230 110) (xy 198.75 110) (xy 198.75 105.652621)
+        (xy 198.5 70.5) (xy 230.5 70.5) (xy 230.5 109.5) (xy 198.5 109.5)
       )
     )
@@
     (polygon
       (pts
-        (xy 230 103.25) (xy 230 110) (xy 215.25 110) (xy 215.25 90.5) (xy 220.75 90.5)
+        (xy 230 103.25) (xy 230 109.5) (xy 215.25 109.5) (xy 215.25 90.5) (xy 220.75 90.5)
         (xy 220.75 94.75) (xy 220.75 103.25)
       )

Commit message: finished initial layout
Parts:
- removed REF** (x4): MOUNTING_HOLE-M3, MOUNTING_HOLE-M3
- added X1: M3 HOLE, ose-audio-labs:MOUNTING_HOLE-M3, F.Cu at (4.00, 36.0)
- added X2: M3 HOLE, ose-audio-labs:MOUNTING_HOLE-M3, F.Cu at (4.00, -36.0)
- added X3: M3 HOLE, ose-audio-labs:MOUNTING_HOLE-M3, F.Cu at (196.0, -36.0)
- added X4: M3 HOLE, ose-audio-labs:MOUNTING_HOLE-M3, F.Cu at (196.0, 36.0)
- C205: footprint ose-audio-labs:35V-LYTIC-7.5-5 -> ose-audio-labs:35V-LYTIC-7.5-5-10snap
- C207: footprint ose-audio-labs:35V-LYTIC-7.5-5-10snap -> ose-audio-labs:35V-LYTIC-7.5-5
- F1: footprint ose-audio-labs:LITTLEFUSE-0PTF0078P -> LITTLEFUSE-0PTF0078P
- J1: footprint ose-audio-labs:PHEONIX_SPT_5-2POS -> PHEONIX_SPT_5-2POS
- SW1: footprint ose-audio-labs:CK_V80212MS02Q-VOLTAGE_SELECTOR -> CK_V80212MS02Q-VOLTAGE_SELECTOR
- U101: footprint PVQFN-N20-new -> PVQFN-N20
- moved C214 184.9 mm to (178.0, 5.30)
- moved C215 180.5 mm to (178.0, 2.55)
- moved C212 174.0 mm to (178.0, 10.8)
- moved C213 171.8 mm to (178.0, 8.05)
- moved C211 163.9 mm to (178.0, 13.6)
- moved C210 163.0 mm to (188.5, 18.7), turned to 180 degrees
- moved C203 151.3 mm to (124.5, 11.5), turned to 90 degrees
- moved C206 147.7 mm to (157.0, 11.5), turned to 90 degrees
- moved C104 142.9 mm to (124.5, -30.0)
- moved R202 138.9 mm to (171.5, 9.50), turned to 270 degrees
- moved C207 133.4 mm to (157.0, 30.0), turned to 90 degrees
- moved LED201 126.4 mm to (171.5, 14.5), turned to 270 degrees
- moved C205 123.8 mm to (140.8, 20.8), turned to 90 degrees
- moved U201 123.2 mm to (182.7, 19.4)
- moved LED101 121.5 mm to (171.5, -14.5), turned to 90 degrees
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Connections:
- J3 pad 1: UNREG-B -> ENABLE-B
- J3 pad 3: ENABLE-B -> UNREG-B
- LED101 pad 2: POS-A -> UNREG-A
- LED201 pad 2: POS-B -> UNREG-B
- U201 pad 10: Net-(SW202-Pad6) -> Net-(SW202-Pad3)
- U201 pad 11: Net-(SW202-Pad7) -> Net-(SW202-Pad2)
- U201 pad 12: Net-(SW202-Pad8) -> Net-(SW202-Pad1)
- U201 pad 4: Net-(SW202-Pad1) -> Net-(SW202-Pad8)
- U201 pad 5: Net-(SW202-Pad2) -> Net-(SW202-Pad7)
- U201 pad 6: Net-(SW202-Pad3) -> Net-(SW202-Pad6)
- U201 pad 8: Net-(SW202-Pad4) -> Net-(SW202-Pad5)
- U201 pad 9: Net-(SW202-Pad5) -> Net-(SW202-Pad4)
Routing:
- net UNREG-B: track 0.00 -> 93.7 mm
- net Net-(C201-Pad2): track 0.00 -> 58.0 mm
- net ENABLE-B: track 0.00 -> 56.1 mm
- net NEG-B: track 0.00 -> 41.9 mm
- net SENSE-B: track 0.00 -> 40.2 mm, vias 0 -> 1
- net Net-(C201-Pad1): track 0.00 -> 31.8 mm
- net UNREG-A: track 106.2 -> 84.6 mm
- net Net-(C202-Pad2): track 0.00 -> 10.9 mm
- net POS-B: track 0.00 -> 9.94 mm
- net NEG-A: track 44.7 -> 54.1 mm
- net Net-(SW202-Pad8): track 0.00 -> 7.37 mm
- net Net-(SW202-Pad1): track 0.00 -> 7.29 mm
- net Net-(SW202-Pad7): track 0.00 -> 5.73 mm
- net Net-(SW202-Pad2): track 0.00 -> 5.62 mm
- net Net-(SW202-Pad5): track 0.00 -> 4.57 mm
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- added copper zone on B.Cu, net NEG-B
- added copper zone on F.Cu, net NEG-B
- added copper zone on F.Cu, net POS-B
- added copper zone on F.Cu, net UNREG-B
