File: oal-psu.kicad_pcb (KiCad board)
At the start: 2 copper layers, 200 x 80 mm, 61 parts, among them J1 MAINS_LINE, J2 MAINS_NEUTRAL, J3 OUTPUT, P101 ENABLE_A, P2 OUTPUT_SELECT, P201 ENABLE_B, SW1 DPDT_SLIDE, SW102 VOLTAGE_A, SW202 VOLTAGE_B, T1 TALEMA 15/25VA, U101 TPS7A4700, U201 TPS7A4700, X1 M3 HOLE, X2 M3 HOLE, X3 M3 HOLE, X4 M3 HOLE

Commit message: layout complete
Parts:
- added X5: M3 HOLE, ose-audio-labs:MOUNTING_HOLE-M3, F.Cu at (180.0, 100.0)
- C108, C208: footprint Capacitors_Tantalum_SMD:TantalC_SizeD_EIA-7343_Reflow -> Capacitors_Tantalum_SMD:TantalC_SizeX_EIA-7343
- D101, D102, D103, D104, D201, D202, D203, D204: footprint ose-audio-labs:DO-221AC -> ose-audio-labs:DO-221AC_SlimSMA
- J1: footprint PHEONIX_SPT_5-2POS -> ose-audio-labs:PHEONIX_SPT_5-2POS
- LED101, LED201: footprint LEDs:LED-1206 -> ose-audio-labs:LED-1206
- SW1: footprint CK_V80212MS02Q-VOLTAGE_SELECTOR -> ose-audio-labs:CK_V80212MS02Q-VOLTAGE_SELECTOR
- SW102, SW202: footprint ose-audio-labs:DIP8-HALF-PITCH -> ose-audio-labs:DIP8-HALF-PITCH-CHS-08B
- moved SW202 108.4 mm to (222.0, 130.0)
- moved C101 107.7 mm to (145.5, 69.5)
- moved C102 107.7 mm to (152.0, 69.5)
- moved C103 107.7 mm to (164.5, 88.5)
- moved C104 107.7 mm to (164.5, 70.0)
- moved C105 107.7 mm to (180.8, 79.2)
- moved C106 107.7 mm to (197.0, 88.5)
- moved C107 107.7 mm to (197.0, 70.0)
- moved C108 107.7 mm to (208.9, 79.1), turned to 180 degrees
- moved C109 107.7 mm to (217.6, 85.3)
- moved C110 107.7 mm to (216.9, 81.5)
- moved C111 107.7 mm to (225.0, 86.2)
- moved C112 107.7 mm to (225.0, 89.0)
- moved C113 107.7 mm to (225.0, 91.8)
- moved C114 107.7 mm to (225.0, 94.5)
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Routing:
- net SENSE-A: track 24.6 -> 33.1 mm
- net UNREG-A: track 84.6 -> 85.6 mm
- net Net-(SW102-Pad4): track 4.51 -> 5.13 mm

Commit message: layout attempt 2
Parts:
- C110: footprint Capacitors_SMD:C_0805 -> C_0805-5mm-FILM
- C113: footprint Capacitors_SMD:C_1206 -> ose-audio-labs:C_1206-FILM-PADS
- moved LED101 11.5 mm to (208.3, 96.6), turned to 180 degrees
- moved P101 7.38 mm to (207.5, 64.0), turned to 90 degrees
- moved C108 6.44 mm to (211.5, 85.0), turned to 90 degrees
- moved R102 6.38 mm to (213.3, 96.6), turned to 180 degrees
- moved C110 5.52 mm to (213.7, 77.0)
- moved U101 3.05 mm to (221.6, 77.8)
- moved C111 3.01 mm to (223.0, 84.0)
- moved C112 2.83 mm to (223.0, 87.0)
- moved C113 2.66 mm to (223.0, 90.0)
- moved C109 2.59 mm to (216.5, 83.0)
- moved C114 2.50 mm to (223.0, 93.0)
- moved C115 2.36 mm to (223.0, 96.0)
- moved SW102 1.86 mm to (221.6, 68.2)
- moved P2 0.56 mm to (229.5, 97.5)
Routing:
- net NEG-A: track 54.2 -> 33.8 mm
- net UNREG-A: track 85.6 -> 92.8 mm
- net Net-(C110-Pad2): track 2.47 -> 6.64 mm
- net SENSE-A: track 33.1 -> 35.6 mm
- net Net-(SW102-Pad4): track 5.13 -> 3.41 mm
- net Net-(SW102-Pad3): track 5.04 -> 3.67 mm
- net Net-(SW102-Pad2): track 6.15 -> 4.84 mm
- net Net-(SW102-Pad1): track 7.80 -> 6.51 mm
- net ENABLE-A: track 67.8 -> 68.8 mm
- net Net-(SW102-Pad7): track 5.77 -> 4.80 mm
- net POS-A: track 5.91 -> 4.95 mm
- net Net-(SW102-Pad6): track 4.52 -> 3.63 mm
- net Net-(SW102-Pad8): track 7.23 -> 6.44 mm

Commit message: beginning new layout for rail b
Parts:
- C210: footprint Capacitors_SMD:C_0805 -> ose-audio-labs:C_0805-5mm-FILM
- C213: footprint Capacitors_SMD:C_1206 -> ose-audio-labs:C_1206-FILM-PADS
- moved SW202 130.6 mm to (181.6, 5.81), turned to 0 degrees
- moved LED201 119.0 mm to (168.5, 3.50), turned to 180 degrees
- moved C210 117.7 mm to (173.7, 14.5), turned to 0 degrees
- moved R202 112.8 mm to (173.0, 3.50), turned to 180 degrees
- moved U201 111.9 mm to (181.6, 15.3), turned to 180 degrees
- moved R102 107.9 mm to (173.0, -3.50)
- moved LED101 107.7 mm to (168.5, -3.50)
- moved C101 107.7 mm to (105.5, -30.5)
- moved C102 107.7 mm to (112.0, -30.5)
- moved C103 107.7 mm to (124.5, -11.5)
- moved C104 107.7 mm to (124.5, -30.0)
- moved C105 107.7 mm to (140.8, -20.8)
- moved C106 107.7 mm to (157.0, -11.5)
- moved C107 107.7 mm to (157.0, -30.0)
- moved C109 107.7 mm to (176.5, -17.0)
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Routing:
- net SENSE-B: track 40.2 -> 0.00 mm, vias 1 -> 0
- net ENABLE-B: track 56.1 -> 33.8 mm
- net NEG-B: track 41.9 -> 23.3 mm
- net UNREG-B: track 94.0 -> 83.0 mm
- net POS-B: track 9.94 -> 4.12 mm
- net Net-(C210-Pad2): track 2.41 -> 6.56 mm
- net Net-(LED201-Pad1): track 2.63 -> 0.00 mm
- net Net-(LED101-Pad1): track 2.63 -> 0.00 mm
- net Net-(SW202-Pad7): track 6.15 -> 4.68 mm
- net Net-(SW202-Pad8): track 7.80 -> 6.34 mm
- net Net-(SW202-Pad6): track 4.98 -> 3.51 mm
- net Net-(SW202-Pad5): track 4.99 -> 3.52 mm
- net Net-(SW202-Pad4): track 4.73 -> 3.29 mm
- net Net-(SW202-Pad3): track 4.48 -> 3.55 mm
- net Net-(SW202-Pad2): track 5.58 -> 4.72 mm
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- removed copper zone on F.Cu, net POS-B

Commit message: layout complete
Parts:
- added REF**: TH-VIA, TH-VIA, F.Cu at (181.5, 4.00)
- moved P201 39.2 mm to (167.5, 4.00), turned to 90 degrees
- moved LED201 32.5 mm to (168.5, 36.0)
- moved R202 32.5 mm to (173.0, 36.0)
- moved LED101 0.50 mm to (168.5, -4.00)
- moved R102 0.50 mm to (173.0, -4.00)
Connections:
- J3 pad 1: ENABLE-B -> UNREG-B
- J3 pad 3: UNREG-B -> ENABLE-B
Routing:
- net SENSE-B: track 0.00 -> 32.2 mm, vias 0 -> 1
- net ENABLE-B: track 33.8 -> 59.5 mm
- net NEG-B: track 23.3 -> 28.7 mm
- net Net-(C201-Pad2): track 58.0 -> 63.1 mm
- net POS-B: track 4.12 -> 8.04 mm
- net Net-(C101-Pad2): track 45.0 -> 48.7 mm
- net UNREG-B: track 83.0 -> 80.7 mm
- net Net-(LED201-Pad1): track 0.00 -> 2.13 mm
- net Net-(LED101-Pad1): track 0.00 -> 2.13 mm
- net Net-(C202-Pad2): track 10.9 -> 11.5 mm
- added copper zone on F.Cu, net POS-B

Commit message: new output connectors
Parts:
- removed J3: OUTPUT, ose-audio-labs:PHEONIX_MC1.5-12-G-3.5
- added P3: UNREG_A, ose-audio-labs:Phoenix-PTSM-0,5-3, F.Cu at (236.0, 83.5)
- added P4: REG_A, ose-audio-labs:Phoenix-PTSM-0,5-3, F.Cu at (236.0, 94.5)
- added P5: REG_B, ose-audio-labs:Phoenix-PTSM-0,5-3, F.Cu at (236.0, 105.5)
- added P6: UNREG_B, ose-audio-labs:Phoenix-PTSM-0,5-3, F.Cu at (236.0, 116.5)
- C113, C213: footprint ose-audio-labs:C_1206-FILM-PADS -> Capacitors_SMD:C_1206
- C114, C212: footprint Capacitors_SMD:C_1206 -> ose-audio-labs:C_1206-FILM-PADS
- moved C101 107.7 mm to (145.5, 69.5)
- moved C102 107.7 mm to (152.0, 69.5)
- moved C103 107.7 mm to (164.5, 88.5)
- moved C104 107.7 mm to (164.5, 70.0)
- moved C105 107.7 mm to (180.8, 79.2)
- moved C106 107.7 mm to (197.0, 88.5)
- moved C107 107.7 mm to (197.0, 70.0)
- moved C108 107.7 mm to (211.5, 85.0)
- moved C109 107.7 mm to (216.5, 83.0)
- moved C110 107.7 mm to (213.7, 77.0)
- moved C111 107.7 mm to (223.0, 84.0)
- moved C112 107.7 mm to (223.0, 87.0)
- moved C113 107.7 mm to (223.0, 90.0)
- moved C114 107.7 mm to (223.0, 93.0)
- moved C115 107.7 mm to (223.0, 96.0)
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Routing:
- net ENABLE-B: track 59.5 -> 65.2 mm
- net ENABLE-A: track 68.8 -> 67.1 mm
- net NEG-B: track 28.7 -> 30.0 mm
- net SENSE-B: track 32.2 -> 30.9 mm

Commit message: layout updates
Parts:
- added G***: LOGO, OAL_logo, F.Cu at (101.0, 0.00)
- added REF**: Symbol_Highvoltage_Type1_CopperTop_Small, Symbol_Highvoltage_Type1_SilkTop, F.Cu at (21.5, 19.5)
- C113, C213: footprint Capacitors_SMD:C_1206 -> ose-audio-labs:C_1206-FILM-PADS
- C114: footprint ose-audio-labs:C_1206-FILM-PADS -> Capacitors_SMD:C_1206
- C214: renamed from C212; footprint ose-audio-labs:C_1206-FILM-PADS -> Capacitors_SMD:C_1206
- T1: footprint ose-audio-labs:TALEMA_70000K_35VA -> TALEMA_70000K_35VA
- moved C203 108.4 mm to (124.5, 10.8)
- moved C204 108.4 mm to (124.5, 29.2)
- moved C205 108.4 mm to (140.8, 20.0)
- moved C206 108.4 mm to (157.0, 10.8)
- moved C207 108.4 mm to (157.0, 29.2)
- moved C101 107.7 mm to (105.5, -30.5)
- moved C102 107.7 mm to (112.0, -30.5)
- moved C108 107.7 mm to (171.5, -15.0)
- moved C109 107.7 mm to (176.5, -17.0)
- moved C110 107.7 mm to (173.7, -23.0)
- moved C111 107.7 mm to (183.0, -16.0)
- moved C112 107.7 mm to (183.0, -13.0)
- moved C113 107.7 mm to (183.0, -10.0)
- moved C114 107.7 mm to (183.0, -7.00)
- moved C115 107.7 mm to (183.0, -4.00)
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- renumbered C215 to C211, C214 to C212, C211 to C215
Connections:
- P3 pad 1: ENABLE-A -> UNREG-A
- P3 pad 3: UNREG-A -> ENABLE-A
- P5 pad 1: SENSE-B -> NEG-B
- P5 pad 2: NEG-B -> POS-B
- P5 pad 3: POS-B -> SENSE-B
Routing:
- net UNREG-A: track 92.9 -> 85.7 mm
- net ENABLE-A: track 67.1 -> 59.9 mm
- net ENABLE-B: track 65.2 -> 60.6 mm
- net UNREG-B: track 80.9 -> 77.3 mm
- net SENSE-B: track 30.9 -> 27.8 mm
Other:
- board text added: "+"
- board text added: "-"
- board text added: "DANGER DANGER HIGH VOLTAGE!"
- board text added: "DANGER DANGER HIGH VOLTAGE! DO NOT TOUCH ANYTHING!"
- board text added: "LINE"
- board text added: "NEUTRAL"
- board text added: "OAL PSU rev A"
- board text added: "Ose Audio Labs 2016"
